File: PCB/TANDY_600_96K_SRAM.kicad_sch (KiCad schematic)
At the start: 5 parts, among them J1 DIN-41612-44-M-RA, U1 628128, U2 74HC148

Commit message: silkscreen, symbols, footprints touchups
Parts:
- J1: value DIN-41612-44-M-RA -> DIN 41612 2x22 male right-angle; footprint 000_LOCAL:DIN41612-44P-male-horiz -> 000_LOCAL:DIN 41612 2x22 male right-angle; symbol 000_LOCAL:DIN41612-44 -> 000_LOCAL:DIN 41612 2x22 male right-angle
- U1: value 628128 -> 628128_SOP; symbol 000_LOCAL:628128_DIP32_SSOP32 -> 000_LOCAL:628128_SOP
Connections:
- net GND: now also J1.S1 (mount), J1.S2 (mount)
Changed lines of the file:
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@@
     (pin "2")
   )
-  (symbol (lib_id "000_LOCAL:DIN41612-44") (at 71.12 76.2 0) (unit 1)
-    (in_bom yes) (on_board yes)
-    (property "Reference" "J1" (id 0) (at 72.39 44.45 0))
-    (property "Value" "DIN-41612-44-M-RA" (id 1) (at 72.39 46.99 0))
-    (property "Footprint" "000_LOCAL:DIN41612-44P-male-horiz" (id 2) (at 71.12 76.2 0)
+  (symbol (lib_id "000_LOCAL:DIN 41612 2x22 male right-angle") (at 71.12 76.2 0) (unit 1)
+    (in_bom yes) (on_board yes)
+    (property "Reference" "J1" (id 0) (at 72.898 39.37 0))
+    (property "Value" "DIN 41612 2x22 male right-angle" (id 1) (at 73.152 42.037 0))
+    (property "Footprint" "000_LOCAL:DIN 41612 2x22 male right-angle" (id 2) (at 71.12 76.2 0)
       (effects (font (size 1.27 1.27)) hide)
     )
@@
     (pin "9A")
     (pin "9B")
+    (pin "S1")
+    (pin "S2")
   )
   (symbol (lib_id "000_LOCAL:VCC") (at 137.16 45.72 0) (unit 1)
@@
     (pin "1")
   )
-  (symbol (lib_id "000_LOCAL:GND") (at 124.46 96.52 0) (unit 1)
-    (in_bom yes) (on_board yes)
-    (property "Reference" "#PWR0126" (id 0) (at 124.46 102.87 0)
-      (effects (font (size 1.27 1.27)) hide)
-    )
-    (property "Value" "GND" (id 1) (at 125.222 101.6 0))
-    (property "Footprint" "" (id 2) (at 124.46 96.52 0)
-      (effects (font (size 1.27 1.27)) hide)
-    )
-    (property "Datasheet" "" (id 3) (at 124.46 96.52 0)
-      (effects (font (size 1.27 1.27)) hide)
-    )
-    (pin "1")
-  )
-  (symbol (lib_id "000_LOCAL:628128_DIP32_SSOP32") (at 180.34 73.66 0) (unit 1)
+  (symbol (lib_id "000_LOCAL:628128_SOP") (at 180.34 73.66 0) (unit 1)
     (in_bom yes) (on_board yes)
     (property "Reference" "U1" (id 0) (at 186.055 46.863 0))
-    (property "Value" "628128" (id 1) (at 186.182 48.895 0))
+    (property "Value" "628128_SOP" (id 1) (at 182.88 50.165 0)
+      (effects (font (size 1.27 1.27)) (justify left bottom))
+    )
     (property "Footprint" "000_LOCAL:SOP-32W" (id 2) (at 180.34 73.66 0)
       (effects (font (size 1.27 1.27)) hide)
@@
     (pin "9")
   )
-  (symbol (lib_id "000_LOCAL:GND") (at 180.34 99.06 0) (unit 1)
-    (in_bom yes) (on_board yes)
-    (property "Reference" "#PWR0127" (id 0) (at 180.34 105.41 0)
-      (effects (font (size 1.27 1.27)) hide)
-    )
-    (property "Value" "GND" (id 1) (at 181.102 104.14 0))
-    (property "Footprint" "" (id 2) (at 180.34 99.06 0)
-      (effects (font (size 1.27 1.27)) hide)
-    )
-    (property "Datasheet" "" (id 3) (at 180.34 99.06 0)
+  (symbol (lib_id "000_LOCAL:GND") (at 72.39 49.53 0) (mirror x) (unit 1)
+    (in_bom yes) (on_board yes)
+    (property "Reference" "#PWR0127" (id 0) (at 72.39 43.18 0)
+      (effects (font (size 1.27 1.27)) hide)
+    )
+    (property "Value" "GND" (id 1) (at 72.39 45.974 0))
+    (property "Footprint" "" (id 2) (at 72.39 49.53 0)
+      (effects (font (size 1.27 1.27)) hide)
+    )
+    (property "Datasheet" "" (id 3) (at 72.39 49.53 0)
+      (effects (font (size 1.27 1.27)) hide)
+    )
+    (pin "1")
+  )
+  (symbol (lib_id "000_LOCAL:GND") (at 72.39 105.41 0) (unit 1)
+    (in_bom yes) (on_board yes)
+    (property "Reference" "#PWR0126" (id 0) (at 72.39 111.76 0)
+      (effects (font (size 1.27 1.27)) hide)
+    )
+    (property "Value" "GND" (id 1) (at 73.152 110.49 0))
+    (property "Footprint" "" (id 2) (at 72.39 105.41 0)
+      (effects (font (size 1.27 1.27)) hide)
+    )
+    (property "Datasheet" "" (id 3) (at 72.39 105.41 0)
       (effects (font (size 1.27 1.27)) hide)
     )
@@
       (reference "#PWR0125") (unit 1) (value "VCC") (footprint "")
     )
-    (path "/00000000-0000-0000-0000-0000613af808"
+    (path "/fe9d6ac1-2102-4d78-bdd3-5f22b011e3c1"
       (reference "#PWR0126") (unit 1) (value "GND") (footprint "")
     )
-    (path "/00000000-0000-0000-0000-00006143edd7"
+    (path "/ee5854f3-4328-4382-bd7b-57b5d7cb8000"
       (reference "#PWR0127") (unit 1) (value "GND") (footprint "")
     )
@@
     )
     (path "/00000000-0000-0000-0000-000061163f2f"
-      (reference "J1") (unit 1) (value "DIN-41612-44-M-RA") (footprint "000_LOCAL:DIN41612-44P-male-horiz")
+      (reference "J1") (unit 1) (value "DIN 41612 2x22 male right-angle") (footprint "000_LOCAL:DIN 41612 2x22 male right-angle")
     )
     (path "/00000000-0000-0000-0000-0000613c8a04"
-      (reference "U1") (unit 1) (value "628128") (footprint "000_LOCAL:SOP-32W")
+      (reference "U1") (unit 1) (value "628128_SOP") (footprint "000_LOCAL:SOP-32W")
     )
     (path "/00000000-0000-0000-0000-0000613445a6"

Commit message: re-visible gnd pins on symbols
Changed lines of the file:
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@@
     (pin "1")
   )
-  (symbol (lib_id "000_LOCAL:GND") (at 111.76 88.9 0) (unit 1)
-    (in_bom yes) (on_board yes)
-    (property "Reference" "#PWR0114" (id 0) (at 111.76 95.25 0)
-      (effects (font (size 1.27 1.27)) hide)
-    )
-    (property "Value" "GND" (id 1) (at 112.268 93.726 0))
+  (symbol (lib_id "000_LOCAL:GND") (at 111.76 88.9 270) (unit 1)
+    (in_bom yes) (on_board yes)
+    (property "Reference" "#PWR0114" (id 0) (at 105.41 88.9 0)
+      (effects (font (size 1.27 1.27)) hide)
+    )
+    (property "Value" "GND" (id 1) (at 106.934 88.9 90))
     (property "Footprint" "" (id 2) (at 111.76 88.9 0)
       (effects (font (size 1.27 1.27)) hide)
@@
     (pin "9")
   )
+  (symbol (lib_id "000_LOCAL:GND") (at 180.34 99.06 0) (unit 1)
+    (in_bom yes) (on_board yes)
+    (property "Reference" "#PWR?" (id 0) (at 180.34 105.41 0)
+      (effects (font (size 1.27 1.27)) hide)
+    )
+    (property "Value" "GND" (id 1) (at 181.102 104.14 0))
+    (property "Footprint" "" (id 2) (at 180.34 99.06 0)
+      (effects (font (size 1.27 1.27)) hide)
+    )
+    (property "Datasheet" "" (id 3) (at 180.34 99.06 0)
+      (effects (font (size 1.27 1.27)) hide)
+    )
+    (pin "1")
+  )
+  (symbol (lib_id "000_LOCAL:GND") (at 124.46 96.52 0) (unit 1)
+    (in_bom yes) (on_board yes)
+    (property "Reference" "#PWR?" (id 0) (at 124.46 102.87 0)
+      (effects (font (size 1.27 1.27)) hide)
+    )
+    (property "Value" "GND" (id 1) (at 125.222 101.6 0))
+    (property "Footprint" "" (id 2) (at 124.46 96.52 0)
+      (effects (font (size 1.27 1.27)) hide)
+    )
+    (property "Datasheet" "" (id 3) (at 124.46 96.52 0)
+      (effects (font (size 1.27 1.27)) hide)
+    )
+    (pin "1")
+  )
   (symbol (lib_id "000_LOCAL:GND") (at 72.39 49.53 0) (mirror x) (unit 1)
     (in_bom yes) (on_board yes)
@@
       (reference "#PWR0127") (unit 1) (value "GND") (footprint "")
     )
+    (path "/10c3d28d-99bc-4b2f-b483-29063755563e"
+      (reference "#PWR?") (unit 1) (value "GND") (footprint "")
+    )
+    (path "/6abd9a4f-c91d-48bb-ad4c-158231fb08b4"
+      (reference "#PWR?") (unit 1) (value "GND") (footprint "")
+    )
     (path "/00000000-0000-0000-0000-0000586e7dab"
