File: PCB/TANDY_600_RAM_THT.kicad_pcb (KiCad board)
At the start: 2 copper layers, 68.6 x 45.1 mm, 7 parts, among them J1 DIN 41612 2x22 male right-ang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, U1 628128_DIP, U2 74HC08

Commit message: tht routing
Routing:
- net /CS2: track 55.7 -> 47.0 mm
- net /~{OE}: track 29.7 -> 21.8 mm, vias 2 -> 0
- net /D2: track 24.7 -> 30.9 mm, vias 2 -> 0
- net /~{CS1_C}: track 46.2 -> 51.4 mm, vias 2 -> 1
- net /D5: track 14.5 -> 10.8 mm, vias 2 -> 0
- net /D3: track 10.3 -> 13.3 mm
- net /A10: track 30.7 -> 28.5 mm, vias 0 -> 2
- net /A13: track 11.2 -> 13.4 mm
- net /A0: track 20.9 -> 22.1 mm
- net /A11: track 19.4 -> 18.4 mm
- net /~{WE}: track 45.5 -> 46.2 mm
- net GND: vias 5 -> 3

Commit message: tht routing
Parts:
- U1: value 628128_DIP -> 628128_SOP
Connections:
- U2 pad 1: /~{CS1_B} -> GND
- U2 pad 10: GND -> /A15
- U2 pad 2: /~{CS1_A} -> GND
- U2 pad 3: /A16 -> unconnected-(U2-Pad3)
- U2 pad 4: /A15 -> /~{CS1_A}
- U2 pad 5: /A16 -> /~{CS1_B}
- U2 pad 6: /~{CS1} -> /A16
- U2 pad 8: unconnected-(U2-Pad8) -> /~{CS1}
- U2 pad 9: GND -> /A16
Routing:
- net /~{CS1_B}: track 57.3 -> 45.9 mm, vias 2 -> 1
- net /~{CS1}: track 29.2 -> 18.4 mm
- net /A15: track 42.0 -> 33.5 mm, vias 2 -> 0
- net /D7: track 6.13 -> 8.23 mm
- net /~{CS1_A}: track 44.2 -> 42.9 mm, vias 2 -> 0
- net /A0: track 22.1 -> 23.0 mm
- net /A11: track 18.4 -> 17.6 mm
- net /A16: track 29.8 -> 30.3 mm, vias 1 -> 0
- net GND: vias 3 -> 0

Commit message: gnd on tiny, new dual sch, bus connector symbol & footprint
Parts:
- U1: value 628128_SOP -> 628128
Routing:
- net /A16: track 30.3 -> 37.0 mm, vias 0 -> 2
- net /~{CS1_A}: track 42.9 -> 48.0 mm, vias 0 -> 1
- net /~{CS1_B}: track 45.9 -> 47.1 mm, vias 1 -> 2
- net /A15: track 33.5 -> 34.7 mm, vias 0 -> 2
- net GND: vias 0 -> 1
Other:
- board text added: "${COMMENT2} ${REVISION}"
- board text added: "a1"
- board text added: "a22"
- board text added: "b1"
- board text added: "b22"
- board text removed: "${COMMENT2} ${TITLE} v${REVISION}"
- board text removed: "22A"
- board text removed: "22B"

Commit message: footprints, ground paths
Parts:
- J1: footprint 000_LOCAL:DIN 41612 2x22 male right-angle -> 000_LOCAL:DIN-41612_02x22_male_horizontal

Commit message: undo accidentally saved filleted tracks on THT
Routing:
- net VMEM: track 11.9 -> 11.2 mm
